File: EliteCSTM32F411.kicad_pcb (KiCad board)
At the start: 2 copper layers, 17.8 x 30.5 mm, 27 parts, among them SW1 Boot Mode, SW2 Reset Switch, U1 STM32F411CEUx, U2 XC6206PxxxMR, U3 Elite-C, Y1 8Mhz 3225

Commit message: redid some pins, i2c compatible with pro micro. (also redid some labels)
Connections:
- U1 pad 20: PB2 -> (no net)
- U1 pad 21: (no net) -> PB10
- U3 pad 10: PB7 -> PB5
- U3 pad 24: PB2 -> PB10
- U3 pad 5: PA15 -> PB6
- U3 pad 6: PB3 -> PB7
- U3 pad 7: PB4 -> PA15
- U3 pad 8: PB5 -> PB3
- U3 pad 9: PB6 -> PB4
Routing:
- net PB10: track 0.00 -> 20.1 mm
- net PB2: track 20.0 -> 0.00 mm
- net PB5: track 4.58 -> 9.33 mm
- net PA15: track 8.06 -> 4.22 mm
- net PB6: track 6.22 -> 9.80 mm, vias 0 -> 1
- net PB4: track 4.63 -> 7.08 mm
- net GND: track 38.1 -> 39.5 mm
- net PB3: track 6.18 -> 4.99 mm
- net PB7: track 8.37 -> 7.93 mm, vias 0 -> 1
Other:
- board text added: "A0"
- board text added: "A1"
- board text added: "A13"
- board text added: "A15"
- board text added: "A2"
- board text added: "A3"
- board text added: "A4"
- board text added: "A5"
- board text added: "A6"
- board text added: "A7"
- board text added: "B0"
- board text added: "B1"
- board text added: "B10"
- board text added: "B3"
- board text added: "B4"
- board text added: "B5"
- board text added: "B6"
- board text added: "B7"
- board text added: "B8"
- board text added: "B9"
- board text added: "C13"
- board text added: "C14"
- board text added: "C15"
- board text added: "D+"
- board text added: "D-"
- board text removed: "PA0"
- board text removed: "PA1"
- board text removed: "PA13"
- board text removed: "PA15"
- board text removed: "PA2"
- board text removed: "PA3"
- board text removed: "PA4"
- board text removed: "PA5"
- board text removed: "PA6"
- board text removed: "PA7"
- board text removed: "PB0"
- board text removed: "PB1"
- board text removed: "PB2"
- board text removed: "PB3"
- board text removed: "PB4"
- board text removed: "PB5"
- board text removed: "PB6"
- board text removed: "PB7"
- board text removed: "PB8"
- board text removed: "PB9"
- board text removed: "PC13"
- board text removed: "PC14"
- board text removed: "PC15"
